Commit message: kinnectconnecté

File: src/motoman/motoman_hc10_support/urdf/hc10.gazebo.xacro (robot description, xacro)
@@ -17,40 +17,41 @@
         <xacro:arm_gazebo link="${prefix}link_6_t"/>
         <xacro:arm_gazebo link="${prefix}tool0"/>
+        <xacro:arm_gazebo link="${prefix}kinect_camera"/>
     </xacro:macro>
+    <gazebo reference="camera_depth_frame">
+        <sensor name="kinect_camera" type="depth">
+            <update_rate>20</update_rate>
+            <camera>
+                <horizontal_fov>1.047198</horizontal_fov>
+                <image>
+                    <width>640</width>
+                    <height>480</height>
+                    <format>B8G8R8</format>
+                </image>
+                <clip>
+                    <near>0.05</near>
+                    <far>3</far>
+                </clip>
+            </camera>
+            <plugin name="kinect_controller" filename="libgazebo_ros_openni_kinect.so">
+            <baseline>0.1</baseline>
+            <alwaysOn>true</alwaysOn>
+            <updateRate>10</updateRate>
+            <cameraName>camera_ir</cameraName>
+            <imageTopicName>/camera/color/image_raw</imageTopicName>
+            <cameraInfoTopicName>/camera/color/camera_info</cameraInfoTopicName>
+            <depthImageTopicName>/camera/depth/image_raw</depthImageTopicName>
+            <depthImageCameraInfoTopicName>/camera/depth/camera_info</depthImageCameraInfoTopicName>
+            <pointCloudTopicName>/camera/depth/points</pointCloudTopicName>
+            <frameName>camera_depth_optical_frame</frameName>
+            <distortion_k1>0.0</distortion_k1>
+            <distortion_k2>0.0</distortion_k2>
+            <distortion_k3>0.0</distortion_k3>
+            <distortion_t1>0.0</distortion_t1>
+            <distortion_t2>0.0</distortion_t2>
+            <pointCloudCutoff>0.16</pointCloudCutoff>
+            <pointCloudCutoffMax>10.0</pointCloudCutoffMax>
+            </plugin>
+        </sensor>
+    </gazebo>
 </robot>
-<gazebo reference="camera_depth_frame">
-    <sensor name="kinect_camera" type="depth">
-        <update_rate>20</update_rate>
-        <camera>
-            <horizontal_fov>1.047198</horizontal_fov>
-            <image>
-                <width>640</width>
-                <height>480</height>
-                <format>B8G8R8</format>
-            </image>
-            <clip>
-                <near>0.05</near>
-                <far>3</far>
-            </clip>
-        </camera>
-        <plugin name="kinect_controller" filename="libgazebo_ros_openni_kinect.so">
-        <baseline>0.1</baseline>
-        <alwaysOn>true</alwaysOn>
-        <updateRate>10</updateRate>
-        <cameraName>camera_ir</cameraName>
-        <imageTopicName>/camera/color/image_raw</imageTopicName>
-        <cameraInfoTopicName>/camera/color/camera_info</cameraInfoTopicName>
-        <depthImageTopicName>/camera/depth/image_raw</depthImageTopicName>
-        <depthImageCameraInfoTopicName>/camera/depth/camera_info</depthImageCameraInfoTopicName>
-        <pointCloudTopicName>/camera/depth/points</pointCloudTopicName>
-        <frameName>camera_depth_optical_frame</frameName>
-        <distortion_k1>0.0</distortion_k1>
-        <distortion_k2>0.0</distortion_k2>
-        <distortion_k3>0.0</distortion_k3>
-        <distortion_t1>0.0</distortion_t1>
-        <distortion_t2>0.0</distortion_t2>
-        <pointCloudCutoff>0.16</pointCloudCutoff>
-        <pointCloudCutoffMax>10.0</pointCloudCutoffMax>
-        </plugin>
-    </sensor>
-</gazebo>

File: src/motoman/motoman_hc10_support/urdf/hc10_macro.xacro (robot description, xacro)
@@ -138,4 +138,5 @@
     </link>
     <link name="${prefix}tool0"/>
+    <link name="${prefix}kinect_camera"/>
     <!-- end of link list -->
     <!-- joint list -->
@@ -199,5 +200,5 @@
     <!-- end of joint list -->
     <!-- ROS base_link to Robot Manufacturer World Coordinates transform -->
-    <link name="${prefix}base" />
+    <link name="${prefix}base"/>
     <joint name="${prefix}base_link-base" type="fixed">
       <origin xyz="0 0 0.275" rpy="0 0 0"/>
@@ -205,4 +206,12 @@
       <child link="${prefix}base"/>
     </joint>
+    <joint name="${prefix}camera_joint" type="fixed">
+      <origin xyz="0.15 -1 0.1" rpy="0 0 1.57"/>
+      <child link ="${prefix}kinect_camera"/>
+      <parent link="${prefix}tool0"/>
+      <axis xyz="0 0 0" rpy="0 0 0"/>
+      <limit effort="10000" velocity="1000"/>
+      <dynamics damping="1.0" friction="1.0"/>
+    </joint>
   </xacro:macro>
 </robot>

Commit message: last commit

File: src/motoman/motoman_hc10_support/urdf/hc10.gazebo.xacro (robot description, xacro)
@@ -19,5 +19,5 @@
         <xacro:arm_gazebo link="${prefix}kinect_camera"/>
     </xacro:macro>
-    <gazebo reference="camera_depth_frame">
+    <gazebo reference="kinect_camera">
         <sensor name="kinect_camera" type="depth">
             <update_rate>20</update_rate>
@@ -44,5 +44,5 @@
             <depthImageCameraInfoTopicName>/camera/depth/camera_info</depthImageCameraInfoTopicName>
             <pointCloudTopicName>/camera/depth/points</pointCloudTopicName>
-            <frameName>camera_depth_optical_frame</frameName>
+            <frameName>kinect_optic</frameName>
             <distortion_k1>0.0</distortion_k1>
             <distortion_k2>0.0</distortion_k2>

File: src/motoman/motoman_hc10_support/urdf/hc10_macro.xacro (robot description, xacro)
@@ -139,4 +139,5 @@
     <link name="${prefix}tool0"/>
     <link name="${prefix}kinect_camera"/>
+    <link name="${prefix}kinect_optic"/>
     <!-- end of link list -->
     <!-- joint list -->
@@ -207,5 +208,5 @@
     </joint>
     <joint name="${prefix}camera_joint" type="fixed">
-      <origin xyz="0.15 -1 0.1" rpy="0 0 1.57"/>
+      <origin xyz="0 0 0.05" rpy="0 -1.57 1.57"/>
       <child link ="${prefix}kinect_camera"/>
       <parent link="${prefix}tool0"/>
@@ -214,4 +215,12 @@
       <dynamics damping="1.0" friction="1.0"/>
     </joint>
+    <joint name="${prefix}optic_joint" type="fixed">
+      <origin xyz="0 0 0" rpy="1.57 0 1.57"/>
+      <child link ="${prefix}kinect_optic"/>
+      <parent link="${prefix}kinect_camera"/>
+      <axis xyz="0 0 0" rpy="0 0 0"/>
+      <limit effort="10000" velocity="1000"/>
+      <dynamics damping="1.0" friction="1.0"/>
+    </joint>
   </xacro:macro>
 </robot>
